File: Hardware/morg_grad_cap.kicad_sch (KiCad schematic)
At the start: 231 parts, among them U1 AZ1117-5.0, U10 AZ1117-5.0, U2 AZ1117-5.0, U3 AZ1117-5.0, U4 AZ1117-5.0, U5 AZ1117-5.0, U6 AZ1117-5.0, U7 AZ1117-5.0, U8 AZ1117-5.0, U9 AZ1117-5.0

Commit message: Finished PCB layout
Parts:
- removed A1: Arduino_Nano_v2.x, Module:Arduino_Nano, symbol MCU_Module:Arduino_Nano_v2.x
- removed C100, C7, C8, C87, C88, C89, C90, C91, C92, C93, C94, C95, C96, C97, C98, C99: 1uF, Capacitor_SMD:C_0603_1608Metric_Pad1.08x0.95mm_HandSolder, symbol Device:C_Small
- removed C109, C110, C111, C112, C113, C114, C115, C116, C117, C118, C119, C120: 10uF, Capacitor_SMD:C_0603_1608Metric_Pad1.08x0.95mm_HandSolder, symbol Device:C_Polarized_US
- removed D100, D85, D86, D87, D88, D89, D90, D91, D92, D93, D94, D95, D96, D97, D98, D99: WS2813B, LED_SMD:LED_WS2812_PLCC6_5.0x5.0mm_P1.6mm, symbol LEDs:WS2813B
- removed U10, U5, U7, U8, U9: AZ1117-5.0, Package_TO_SOT_SMD:SOT-223-3_TabPin2, symbol Regulator_Linear:AZ1117-5.0
- added C87, C88, C89, C90, C91, C92, C93: 10uF, Capacitor_SMD:C_0805_2012Metric_Pad1.18x1.45mm_HandSolder, symbol Device:C_Polarized_US
- added H1, H2, H3, H4: MountingHole_Pad, MountingHole:MountingHole_3.2mm_M3_Pad, symbol Mechanical:MountingHole_Pad
- added J1: JST-PH Batt Power In, Connector_JST:JST_PH_S2B-PH-K_1x02_P2.00mm_Horizontal, symbol Connector_Generic:Conn_01x02
- added J2: JST-PH SPI, Connector_JST:JST_PH_S5B-PH-K_1x05_P2.00mm_Horizontal, symbol Connector_Generic:Conn_01x05
- added J3: JST-PH UART/I2C, Connector_JST:JST_PH_S6B-PH-K_1x06_P2.00mm_Horizontal, symbol Connector_Generic:Conn_01x06
- added J4: JST-PH A#, Connector_JST:JST_PH_S6B-PH-K_1x06_P2.00mm_Horizontal, symbol Connector_Generic:Conn_01x06
- added J5: Data Out, Connector_JST:JST_PH_S2B-PH-K_1x02_P2.00mm_Horizontal, symbol Connector_Generic:Conn_01x02
- added R1, R2: 220Ω, Resistor_SMD:R_0603_1608Metric_Pad0.98x0.95mm_HandSolder, symbol Device:R_Small_US
- added U5: QTPy SAMD21, New_Library:Py_QT_SAMD21, symbol New_Library:QT_Py_SAMD21
- C1: renamed from C101; footprint Capacitor_SMD:C_0603_1608Metric_Pad1.08x0.95mm_HandSolder -> Capacitor_SMD:C_0805_2012Metric_Pad1.18x1.45mm_HandSolder
- C103, C104, C105, C106, C107, C108: footprint Capacitor_SMD:C_0603_1608Metric_Pad1.08x0.95mm_HandSolder -> Capacitor_SMD:C_0805_2012Metric_Pad1.18x1.45mm_HandSolder
- C2: renamed from C102; footprint Capacitor_SMD:C_0603_1608Metric_Pad1.08x0.95mm_HandSolder -> Capacitor_SMD:C_0805_2012Metric_Pad1.18x1.45mm_HandSolder
- renumbered C1 to C3, C2 to C4, C3 to C5, C4 to C6, C5 to C7, C6 to C8
Connections:
- net GND: now also C87.2, C88.2, C89.2, C90.2, C91.2, C92.2, C93.2, H1.1, H2.1, H3.1, H4.1, J1.2 (Pin_2), J2.5 (Pin_5), J3.6 (Pin_6), J4.6 (Pin_6), J5.2 (Pin_2), U5.13 (GND)
- net Supply_Rail_5V_U4: now reaches D71.2 (VCC), D72.2 (VCC), D73.2 (VCC), D74.2 (VCC), D75.2 (VCC), D76.2 (VCC), D77.2 (VCC), D78.2 (VCC), D79.2 (VCC), D80.2 (VCC)
- net Supply_Rail_5V_U4: now also C108.1, C61.1, C62.1, C63.1, C64.1, C65.1, C66.1, C67.1, C68.1, C69.1, C70.1, C71.1, C72.1, C73.1, C74.1, C75.1, C76.1, C77.1, C78.1, C79.1, C80.1, C81.1, C82.1, C83.1, C84.1, C85.1, C86.1, D59.2 (VCC), D60.2 (VCC), D61.2 (VCC), D62.2 (VCC), D63.2 (VCC), D64.2 (VCC), D65.2 (VCC), D66.2 (VCC), D67.2 (VCC), D68.2 (VCC), D69.2 (VCC), D70.2 (VCC), D81.2 (VCC), D82.2 (VCC), D83.2 (VCC), D84.2 (VCC), U4.2 (VO), C90.1
- net at D34.3 (DO), D35.4 (DIN): no longer D34.1 (BO), D35.6 (BIN)
- net Supply_Rail_5V_U2: now reaches D31.2 (VCC), D32.2 (VCC), D33.2 (VCC), D34.2 (VCC), D35.2 (VCC), D36.2 (VCC), D37.2 (VCC), D38.2 (VCC), D39.2 (VCC)
- net Supply_Rail_5V_U2: now also C104.1, C22.1, C23.1, C24.1, C25.1, C26.1, C27.1, C28.1, C29.1, C30.1, C31.1, C32.1, C33.1, C34.1, C35.1, C36.1, C37.1, C38.1, C39.1, C40.1, C41.1, D20.2 (VCC), D21.2 (VCC), D22.2 (VCC), D23.2 (VCC), D24.2 (VCC), D25.2 (VCC), D26.2 (VCC), D27.2 (VCC), D28.2 (VCC), D29.2 (VCC), D30.2 (VCC), U2.2 (VO), C88.1; no longer C108.1, D40.2 (VCC), U4.2 (VO)
- net at D33.1 (BO), D34.6 (BIN): no longer D33.3 (DO), D34.4 (DIN)
- net at D49.1 (BO), D50.6 (BIN): no longer D49.3 (DO), D50.4 (DIN)
- net Supply_Rail_5V_U3: now reaches D41.2 (VCC), D42.2 (VCC), D43.2 (VCC), D44.2 (VCC), D45.2 (VCC), D46.2 (VCC), D47.2 (VCC), D48.2 (VCC), D49.2 (VCC), D50.2 (VCC)
- net Supply_Rail_5V_U3: now also C106.1, C42.1, C43.1, C44.1, C45.1, C46.1, C47.1, C48.1, C49.1, C50.1, C51.1, C52.1, C53.1, C54.1, C55.1, C56.1, C57.1, C58.1, C59.1, C60.1, D40.2 (VCC), D51.2 (VCC), D52.2 (VCC), D53.2 (VCC), D54.2 (VCC), D55.2 (VCC), D56.2 (VCC), D57.2 (VCC), D58.2 (VCC), U3.2 (VO), C89.1
- net at D48.3 (DO), D49.4 (DIN): no longer D48.1 (BO), D49.6 (BIN)
- net at D26.3 (DO), D27.4 (DIN): no longer D26.1 (BO), D27.6 (BIN)
- net at D25.3 (DO), D26.4 (DIN): no longer D25.1 (BO), D26.6 (BIN)
- net at D17.1 (BO), D18.6 (BIN): no longer D17.3 (DO), D18.4 (DIN)
- net Supply_Rail_5V_U1: now reaches D11.2 (VCC), D12.2 (VCC), D13.2 (VCC), D14.2 (VCC), D15.2 (VCC), D16.2 (VCC), D17.2 (VCC), D18.2 (VCC), D19.2 (VCC)
- net Supply_Rail_5V_U1: now also C10.1, C11.1, C12.1, C13.1, C14.1, C15.1, C16.1, C17.1, C18.1, C19.1, C2.1, C20.1, C21.1, C3.1, C4.1, C5.1, C6.1, C7.1, C8.1, C9.1, D1.2 (VCC), D10.2 (VCC), D2.2 (VCC), D3.2 (VCC), D4.2 (VCC), D5.2 (VCC), D6.2 (VCC), D7.2 (VCC), D8.2 (VCC), D9.2 (VCC), U1.2 (VO), C87.1; no longer C104.1, D20.2 (VCC), U2.2 (VO)
- net at D16.1 (BO), D17.6 (BIN): no longer D16.3 (DO), D17.4 (DIN)
- net at D39.1 (BO), D40.6 (BIN): no longer D39.3 (DO), D40.4 (DIN)
- net at D38.1 (BO), D39.6 (BIN): no longer D38.3 (DO), D39.4 (DIN)
- net at D32.1 (BO), D33.6 (BIN): no longer D32.3 (DO), D33.4 (DIN)
- net at D31.3 (DO), D32.4 (DIN): no longer D31.1 (BO), D32.6 (BIN)
- net +12V: now reaches C1.1, U1.3 (VI)
- net +12V: now also C103.1, C105.1, C107.1, U2.3 (VI), U3.3 (VI), U4.3 (VI), U6.3 (VI), C91.1, J1.1 (Pin_1)
- net at D30.1 (BO): now also D31.6 (BIN)
- net at D30.3 (DO): now also D31.4 (DIN)
- net at D29.3 (DO), D30.4 (DIN): no longer D29.1 (BO), D30.6 (BIN)
- net at D44.3 (DO), D45.4 (DIN): no longer D44.1 (BO), D45.6 (BIN)
- net at D43.3 (DO), D44.4 (DIN): no longer D43.1 (BO), D44.6 (BIN)
- net at D52.3 (DO), D53.4 (DIN): no longer D52.1 (BO), D53.6 (BIN)
- net at D51.1 (BO), D52.6 (BIN): no longer D51.3 (DO), D52.4 (DIN)
- net at D19.3 (DO), D20.4 (DIN): no longer D19.1 (BO), D20.6 (BIN)
- net at D18.3 (DO), D19.4 (DIN): no longer D18.1 (BO), D19.6 (BIN)
- net at D24.1 (BO), D25.6 (BIN): no longer D24.3 (DO), D25.4 (DIN)
- net at D23.3 (DO), D24.4 (DIN): no longer D23.1 (BO), D24.6 (BIN)
- net at D36.1 (BO), D37.6 (BIN): no longer D36.3 (DO), D37.4 (DIN)
- net at D35.1 (BO), D36.6 (BIN): no longer D35.3 (DO), D36.4 (DIN)
- net at D84.1 (BO), D84.3 (DO): now also R2.1
- net at D8.1 (BO), D9.6 (BIN): no longer D8.3 (DO), D9.4 (DIN)
- net at D7.1 (BO), D8.6 (BIN): no longer D7.3 (DO), D8.4 (DIN)
- net at D13.1 (BO), D14.6 (BIN): no longer D13.3 (DO), D14.4 (DIN)
- net at D12.3 (DO), D13.4 (DIN): no longer D12.1 (BO), D13.6 (BIN)
- net at D11.1 (BO), D12.6 (BIN): no longer D11.3 (DO), D12.4 (DIN)
- net at D10.3 (DO), D11.4 (DIN): no longer D10.1 (BO), D11.6 (BIN)
- net at D6.3 (DO), D7.4 (DIN): no longer D6.1 (BO), D7.6 (BIN)
- net at D22.3 (DO), D23.4 (DIN): no longer D22.1 (BO), D23.6 (BIN)
- net at D21.1 (BO), D22.6 (BIN): no longer D21.3 (DO), D22.4 (DIN)
- net at D54.1 (BO), D55.6 (BIN): no longer D54.3 (DO), D55.4 (DIN)
- net at D53.3 (DO), D54.4 (DIN): no longer D53.1 (BO), D54.6 (BIN)
- net at D58.1 (BO), D59.6 (BIN): no longer D58.3 (DO), D59.4 (DIN)
- net at D57.3 (DO), D58.4 (DIN): no longer D57.1 (BO), D58.6 (BIN)
- net at D10.6 (BIN), D9.1 (BO): no longer D10.4 (DIN), D9.3 (DO)
- net at D20.3 (DO): now also D21.4 (DIN); no longer D20.1 (BO)
- net at D46.3 (DO), D47.4 (DIN): no longer D46.1 (BO), D47.6 (BIN)
- net at D45.1 (BO), D46.6 (BIN): no longer D45.3 (DO), D46.4 (DIN)
- net at D15.3 (DO), D16.4 (DIN): no longer D15.1 (BO), D16.6 (BIN)
- net at D14.3 (DO), D15.4 (DIN): no longer D14.1 (BO), D15.6 (BIN)
- net at D81.3 (DO), D82.4 (DIN): no longer D81.1 (BO), D82.6 (BIN)
- net at D28.3 (DO), D29.4 (DIN): no longer D28.1 (BO), D29.6 (BIN)
- net at D27.1 (BO), D28.6 (BIN): no longer D27.3 (DO), D28.4 (DIN)
- net at D42.1 (BO), D43.6 (BIN): no longer D42.3 (DO), D43.4 (DIN)
- net at D59.3 (DO), D60.4 (DIN): no longer D59.1 (BO), D60.6 (BIN)
- net at D82.1 (BO), D83.6 (BIN): no longer D82.3 (DO), D83.4 (DIN)
- net at D37.3 (DO), D38.4 (DIN): no longer D37.1 (BO), D38.6 (BIN)
- net at D41.1 (BO), D42.6 (BIN): no longer D41.3 (DO), D42.4 (DIN)
- net at D47.1 (BO), D48.6 (BIN): no longer D47.3 (DO), D48.4 (DIN)
- net at D55.3 (DO), D56.4 (DIN): no longer D55.1 (BO), D56.6 (BIN)
- net at D5.3 (DO), D6.4 (DIN): no longer D5.1 (BO), D6.6 (BIN)
- net at D56.3 (DO), D57.4 (DIN): no longer D56.1 (BO), D57.6 (BIN)
- net at D2.1 (BO), D3.6 (BIN): no longer D2.3 (DO), D3.4 (DIN)
- net at D1.3 (DO), D2.4 (DIN): no longer D1.1 (BO), D2.6 (BIN)
- net at D3.3 (DO), D4.4 (DIN): no longer D3.1 (BO), D4.6 (BIN)
- net at D83.3 (DO), D84.4 (DIN): no longer D83.1 (BO), D84.6 (BIN)
- net at D4.1 (BO), D5.6 (BIN): no longer D4.3 (DO), D5.4 (DIN)
- net at D1.4 (DIN): now also D1.6 (BIN), R1.2
- removed net +5V: C10.1, C11.1, C12.1, C13.1, C14.1, C15.1, C16.1, C17.1, C18.1, C19.1, C20.1, C21.1, C22.1, C23.1, C24.1, C25.1, C26.1, C27.1, C28.1, C29.1, C3.1, C30.1, C31.1, C32.1, C33.1, C34.1, C35.1, C36.1, C37.1, C38.1, C39.1, C4.1, C40.1, C41.1, C42.1, C43.1, C44.1, C45.1, C46.1, C47.1, C48.1, C49.1, C5.1, C50.1, C51.1, C52.1, C53.1, C54.1, C55.1, C56.1, C57.1, C58.1, C59.1, C6.1, C60.1, C61.1, C62.1, C63.1, C64.1, C65.1, C66.1, C67.1, C68.1, C69.1, C7.1, C70.1, C71.1, C72.1, C73.1, C74.1, C75.1, C76.1, C77.1, C78.1, C79.1, C8.1, C80.1, C81.1, C82.1, C83.1, C84.1, C85.1, C86.1, C9.1
- new net: D67.1 (BO), D68.6 (BIN)
- new net: D67.3 (DO), D68.4 (DIN)
- new net: D66.3 (DO), D67.4 (DIN)
- new net: D66.1 (BO), D67.6 (BIN)
- new net: D4.3 (DO), D5.4 (DIN)
- new net: D3.1 (BO), D4.6 (BIN)
- new net: D61.1 (BO), D62.6 (BIN)
- new net: D61.3 (DO), D62.4 (DIN)
- new net: D60.3 (DO), D61.4 (DIN)
- new net: D60.1 (BO), D61.6 (BIN)
- new net: D45.3 (DO), D46.4 (DIN)
- new net: D44.1 (BO), D45.6 (BIN)
- new net: D63.1 (BO), D64.6 (BIN)
- new net: D63.3 (DO), D64.4 (DIN)
- new net: D62.3 (DO), D63.4 (DIN)
- new net: D62.1 (BO), D63.6 (BIN)
- new net: D32.3 (DO), D33.4 (DIN)
- new net: D31.1 (BO), D32.6 (BIN)
- new net: D21.3 (DO), D22.4 (DIN)
- new net: D20.1 (BO), D21.6 (BIN)
- new net: D33.3 (DO), D34.4 (DIN)
- new net: D59.1 (BO), D60.6 (BIN)
- new net: D82.3 (DO), D83.4 (DIN)
- new net: D81.1 (BO), D82.6 (BIN)
- new net: D16.3 (DO), D17.4 (DIN)
- new net: D15.1 (BO), D16.6 (BIN)
- new net: D76.1 (BO), D77.6 (BIN)
- new net: D76.3 (DO), D77.4 (DIN)
- new net: D75.3 (DO), D76.4 (DIN)
- new net: D75.1 (BO), D76.6 (BIN)
- new net: D38.3 (DO), D39.4 (DIN)
- new net: D37.1 (BO), D38.6 (BIN)
- new net: D47.3 (DO), D48.4 (DIN)
- new net: D46.1 (BO), D47.6 (BIN)
- new net: D58.3 (DO), D59.4 (DIN)
- new net: D57.1 (BO), D58.6 (BIN)
- new net: D83.1 (BO), D84.6 (BIN)
- new net: D14.1 (BO), D15.6 (BIN)
- new net: D35.3 (DO), D36.4 (DIN)
- new net: D34.1 (BO), D35.6 (BIN)
- new net: D41.3 (DO), D42.4 (DIN)
- new net: D40.3 (DO), D41.4 (DIN)
- new net: D40.1 (BO), D41.6 (BIN)
- new net: D80.1 (BO), D81.6 (BIN)
- new net: D80.3 (DO), D81.4 (DIN)
- new net: D79.3 (DO), D80.4 (DIN)
- new net: D79.1 (BO), D80.6 (BIN)
- new net: D49.3 (DO), D50.4 (DIN)
- new net: D48.1 (BO), D49.6 (BIN)
- new net: D78.3 (DO), D79.4 (DIN)
- new net: D78.1 (BO), D79.6 (BIN)
- new net: D36.3 (DO), D37.4 (DIN)
- new net: D7.3 (DO), D8.4 (DIN)
- new net: D6.1 (BO), D7.6 (BIN)
- new net: D2.3 (DO), D3.4 (DIN)
- new net: D1.1 (BO), D2.6 (BIN)
- new net: D73.1 (BO), D74.6 (BIN)
- new net: D73.3 (DO), D74.4 (DIN)
- new net: D72.3 (DO), D73.4 (DIN)
- new net: D72.1 (BO), D73.6 (BIN)
- new net: D27.3 (DO), D28.4 (DIN)
- new net: D26.1 (BO), D27.6 (BIN)
- new net: D56.1 (BO), D57.6 (BIN)
- new net: D74.3 (DO), D75.4 (DIN)
- new net: D74.1 (BO), D75.6 (BIN)
- new net: J5.1 (Pin_1), R2.2
- new net: D39.3 (DO), D40.4 (DIN)
- new net: D19.1 (BO), D20.6 (BIN)
- new net: D13.3 (DO), D14.4 (DIN)
- new net: D12.1 (BO), D13.6 (BIN)
- new net: D42.3 (DO), D43.4 (DIN)
- new net: D5.1 (BO), D6.6 (BIN)
- new net: D8.3 (DO), D9.4 (DIN)
- new net: D29.1 (BO), D30.6 (BIN)
- new net: D51.3 (DO), D52.4 (DIN)
- new net: D50.3 (DO), D51.4 (DIN)
- new net: D50.1 (BO), D51.6 (BIN)
- new net: D11.3 (DO), D12.4 (DIN)
- new net: D10.1 (BO), D11.6 (BIN)
- new net: D10.4 (DIN), D9.3 (DO)
- new net: D71.3 (DO), D72.4 (DIN)
- new net: D71.1 (BO), D72.6 (BIN)
- new net: D28.1 (BO), D29.6 (BIN)
- new net: D70.3 (DO), D71.4 (DIN)
- new net: D70.1 (BO), D71.6 (BIN)
- new net: D18.1 (BO), D19.6 (BIN)
- new net: D54.3 (DO), D55.4 (DIN)
- new net: D53.1 (BO), D54.6 (BIN)
- new net: D69.1 (BO), D70.6 (BIN)
- new net: D69.3 (DO), D70.4 (DIN)
- new net: D68.3 (DO), D69.4 (DIN)
- new net: D68.1 (BO), D69.6 (BIN)
- new net: D17.3 (DO), D18.4 (DIN)
- new net: D24.3 (DO), D25.4 (DIN)
- new net: D23.1 (BO), D24.6 (BIN)
- new net: D77.3 (DO), D78.4 (DIN)
- new net: D77.1 (BO), D78.6 (BIN)
- new net: D25.1 (BO), D26.6 (BIN)
- new net: D22.1 (BO), D23.6 (BIN)
- new net: D55.1 (BO), D56.6 (BIN)
- new net: D43.1 (BO), D44.6 (BIN)
- new net: D52.1 (BO), D53.6 (BIN)
- new net: D64.1 (BO), D65.6 (BIN)
- new net: D64.3 (DO), D65.4 (DIN)
- new net: D65.3 (DO), D66.4 (DIN)
- new net: D65.1 (BO), D66.6 (BIN)
- new net SAMD_A0: J4.2 (Pin_2), U5.1 (A0)
- new net SAMD_A1: J4.3 (Pin_3), U5.2 (A1)
- new net SAMD_A2: J4.4 (Pin_4), R1.1, U5.3 (A2)
- new net SAMD_A3: J4.5 (Pin_5), U5.4 (A3)
- new net SAMD_MISO: J2.3 (Pin_3), U5.10 (MI)
- new net SAMD_MOSI: J2.4 (Pin_4), U5.11 (MO)
- new net SAMD_RX: J3.5 (Pin_5), U5.8 (RX)
- new net SAMD_SCK: J2.2 (Pin_2), U5.9 (SCK)
- new net SAMD_SCL: J3.3 (Pin_3), U5.6 (SCL)
- new net SAMD_SDA: J3.2 (Pin_2), U5.5 (SDA)
- new net SAMD_TX: J3.4 (Pin_4), U5.7 (TX)
- new net Supply_Rail_5V_U6: C92.1, C93.1, J2.1 (Pin_1), J3.1 (Pin_1), J4.1 (Pin_1), U5.14 (5V), U6.2 (VO)
Other:
- note added: "Each LED: 16mA + 16mA + 16mA = 48mA (R) (G) (B) 7*6 + 6*7 = 84 LEDs 84*48mA = 4,032mA"
- note added: "Max Input Voltage: 18V Configured Output Voltage: 5V Max Output Current: 1,350mA 5V * 4,032mA = 20.16W Consumed 24W/12V = 1.68A Input"
- note removed: "Each LED: 16mA + 16mA + 16mA = 48mA (R) (G) (B) 10*10 = 100 LEDs 100*48mA = 4,800mA"
- note removed: "Max Input Voltage: 18V Configured Output Voltage: 5V Max Output Current: 1,350mA 5V * 4,800mA = 24W Consumed 24W/12V = 2A Input"
- moved on the sheet: C1, C2, C3, C4, C5, C6, C7, C8, U1

Commit message: Added image of schematic
Other:
- company: (none) -> Thomas Francois KXØSTL
- title: (none) -> Mogan Grad Cap
Changed lines of the file:
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@@
 (kicad_sch
-	(version 20231120)
+	(version 20250114)
 	(generator "eeschema")
-	(generator_version "8.0")
+	(generator_version "9.0")
 	(paper "C")
+	(title_block
+		(title "Mogan Grad Cap")
+		(date "2024-12-13")
+		(rev "A")
+		(company "Thomas Francois KXØSTL")
+	)
+	(text "Each LED: 16mA + 16mA + 16mA = 48mA\n            (R)      (G)      (B)\n\n7*6 + 6*7 = 84 LEDs\n\n84*48mA = 4,032mA"
+		(exclude_from_sim no)
+		(at 25.4 413.258 0)
+		(effects
+			(font
+				(size 5.08 5.08)
+			)
+			(justify left bottom)
+		)
+	)
+	(text "Max Input Voltage: 18V\nConfigured Output Voltage: 5V\nMax Output Current: 1,350mA\n5V * 4,032mA = 20.16W Consumed\n24W/12V = 1.68A Input"
+		(exclude_from_sim no)
+		(at 240.792 415.798 0)
+		(effects
+			(font
+				(size 5.08 5.08)
+			)
+			(justify left bottom)
+		)
+	)
+	(text "AZ1117-5.0"
+		(exclude_from_sim no)
+		(at 240.284 371.602 0)
+		(effects
+			(font
+				(size 5.08 5.08)
+				(thickness 1.016)
+				(bold yes)
+			)
+			(justify left bottom)
+		)
+	)
 	(junction
 		(at 378.46 307.34)
@@
 		)
 	)
-	(text "Each LED: 16mA + 16mA + 16mA = 48mA\n            (R)      (G)      (B)\n\n7*6 + 6*7 = 84 LEDs\n\n84*48mA = 4,032mA"
-		(exclude_from_sim no)
-		(at 25.4 413.258 0)
-		(effects
-			(font
-				(size 5.08 5.08)
-			)
-			(justify left bottom)
-		)
-	)
-	(text "Max Input Voltage: 18V\nConfigured Output Voltage: 5V\nMax Output Current: 1,350mA\n5V * 4,032mA = 20.16W Consumed\n24W/12V = 1.68A Input"
-		(exclude_from_sim no)
-		(at 240.792 415.798 0)
-		(effects
-			(font
-				(size 5.08 5.08)
-			)
-			(justify left bottom)
-		)
-	)
-	(text "AZ1117-5.0"
-		(exclude_from_sim no)
-		(at 240.284 371.602 0)
-		(effects
-			(font
-				(size 5.08 5.08)
-				(thickness 1.016)
-				(bold yes)
-			)
-			(justify left bottom)
-		)
-	)
 	(label "Supply_Rail_5V_U1"
 		(at 166.37 33.02 0)
-		(fields_autoplaced yes)
 		(effects
 			(font
@@
 	(label "SAMD_A3"
 		(at 124.46 78.74 180)
-		(fields_autoplaced yes)
 		(effects
 			(font
@@
 	(label "SAMD_MOSI"
 		(at 88.9 76.2 180)
-		(fields_autoplaced yes)
 		(effects
 			(font
@@
 	(label "SAMD_SCK"
 		(at 146.05 62.23 180)
-		(fields_autoplaced yes)
 		(effects
 			(font
@@
 	(label "SAMD_A3"
 		(at 163.83 64.77 0)
-		(fields_autoplaced yes)
 		(effects
 			(font
@@
 	(label "Supply_Rail_5V_U2"
 		(at 166.37 101.6 0)
-		(fields_autoplaced yes)
 		(effects
 			(font
@@
 	(label "SAMD_A2"
 		(at 124.46 76.2 180)
-		(fields_autoplaced yes)
 		(effects
 			(font
@@
 	(label "SAMD_SDA"
 		(at 102.87 71.12 0)
-		(fields_autoplaced yes)
 		(effects
 			(font
@@
 	(label "SAMD_SCL"
 		(at 102.87 73.66 0)
-		(fields_autoplaced yes)
 		(effects
 			(font
@@
 	(label "SAMD_A2"
 		(at 163.83 62.23 0)
-		(fields_autoplaced yes)
 		(effects
 			(font
@@
 	(label "SAMD_SDA"
 		(at 163.83 69.85 0)
-		(fields_autoplaced yes)
 		(effects
 			(font
@@
 	(label "SAMD_A1"
 		(at 163.83 59.69 0)
-		(fields_autoplaced yes)
 		(effects
 			(font
@@
 	(label "SAMD_MISO"
 		(at 146.05 59.69 180)
-		(fields_autoplaced yes)
 		(effects
 			(font
@@
 	(label "SAMD_A1"
 		(at 124.46 73.66 180)
-		(fields_autoplaced yes)
 		(effects
 			(font
@@
 	(label "SAMD_TX"
 		(at 146.05 69.85 180)
-		(fields_autoplaced yes)
 		(effects
 			(font
@@
 	(label "SAMD_TX"
 		(at 102.87 76.2 0)
-		(fields_autoplaced yes)
 		(effects
 			(font
@@
 	(label "SAMD_RX"
 		(at 146.05 72.39 180)
-		(fields_autoplaced yes)
 		(effects
 			(font
@@
 	(label "SAMD_MISO"
 		(at 88.9 73.66 180)
-		(fields_autoplaced yes)
 		(effects
 			(font
@@
 	(label "SAMD_SCK"
 		(at 88.9 71.12 180)
-		(fields_autoplaced yes)
 		(effects
 			(font
@@
 	(label "Supply_Rail_5V_U6"
 		(at 67.31 50.8 0)
-		(fields_autoplaced yes)
 		(effects
 			(font
@@
 	(label "Supply_Rail_5V_U3"
 		(at 166.37 170.18 0)
-		(fields_autoplaced yes)
 		(effects
 			(font
@@
 	(label "SAMD_RX"
 		(at 102.87 78.74 0)
-		(fields_autoplaced yes)
 		(effects
 			(font
@@
 	(label "SAMD_MOSI"
 		(at 146.05 57.15 180)
-		(fields_autoplaced yes)
 		(effects
 			(font
@@
 	(label "SAMD_A0"
 		(at 163.83 57.15 0)
-		(fields_autoplaced yes)
 		(effects
 			(font
@@
 	(label "Supply_Rail_5V_U4"
 		(at 166.37 238.76 0)
-		(fields_autoplaced yes)
 		(effects
 			(font
@@
 	(label "SAMD_SCL"
 		(at 163.83 72.39 0)
-		(fields_autoplaced yes)
 		(effects
 			(font
@@
 	(label "SAMD_A0"
 		(at 124.46 71.12 180)
-		(fields_autoplaced yes)
 		(effects
 			(font
@@
 		)
 	)
+	(embedded_fonts no)
 )
