File: Hardware/Grad/ESP32_MASTER.kicad_sch (KiCad schematic)
At the start: 11 parts, among them J301 Conn_01x40, U101 ESP32-S3-WROOM-1, U103 LM66200DRLR, U201 THVD1400D, U202 TLV75733PDRV

Commit message: Schematic feels done now
Parts:
- added C201: 1uF, New_Library:Worthington_C_0603, symbol Device:C_Polarized_Small_US
- added C202, C204, C215: 22uF, New_Library:Worthington_C_0603, symbol Device:C_Polarized_Small_US
- added C205, C207, C209, C211, C213, C214, C216: 100nF, New_Library:Worthington_C_0402, symbol Device:C_Small_US
- added C212: 22uF, New_Library:Worthington_D_0603, symbol Device:C_Polarized_Small_US
- added D202, D203, D204, D205: RED, New_Library:Worthington_LED_0603, symbol Device:LED_Small
- added L201: 22uH, New_Library:CDRH5D28, symbol Device:L
- added R202: 10, Resistor_SMD:R_1210_3225Metric, symbol Device:R_Small_US
- added RN201: 10k, New_Library:RESCAXE80P320X160X70-8N, symbol Libraries:R_Network04_Split
- added RN202: 430, New_Library:RESCAXE80P320X160X70-8N, symbol Libraries:R_Network04_Split
- added U203: SN74LVC1G139, Package_SO:VSSOP-8_2.3x2mm_P0.5mm, symbol 74xGxx:74LVC1G139
- added U205: TC7MBL3126CFT, Package_SO:TSSOP-14_4.4x5mm_P0.65mm, symbol Analog_Switch:CD4066BPW
- added U206: AP3019AKTTR, Package_TO_SOT_SMD:TSOT-23-6, symbol Driver_LED:AP3019AKTTR
- added U207: W25Q128JVP, Package_SON:WSON-8-1EP_6x5mm_P1.27mm_EP3.4x4.3mm, symbol Memory_Flash:W25Q128JVP
- C203: renamed from C204; footprint (none) -> New_Library:Worthington_C_0603
- C206: renamed from C202; value 47uF -> 22uF; footprint (none) -> New_Library:Worthington_C_0603
- C208: renamed from C201; footprint (none) -> New_Library:Worthington_C_0402
- C210: renamed from C203; footprint (none) -> New_Library:Worthington_C_0402
- D201: footprint (none) -> New_Library:Worthington_LED_0603
- J201: renamed from J301; value Conn_01x40 -> Amphenol 40-Pin FPC; footprint (none) -> New_Library:AMPHENOL_62684-402100ALF; DigiKey (none) -> https://www.digikey.com/en/products/detail/amphenol-cs-fci/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; DigiKey Part (none) -> 62684-402100ALF
- R201: value R_Small_US -> 430; footprint (none) -> New_Library:Worthington_R_0402
- U201: renamed from U103; DigiKey (none) -> https://www.digikey.com/en/products/detail/texas-instrument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; DigiKey Part (none) -> 296-LM66200DRLRCT-ND
- U202: DigiKey (none) -> https://www.digikey.com/en/products/detail/texas-instrument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; DigiKey Part (none) -> 296-50414-1-ND
- U204: renamed from U101; value ESP32-S3-WROOM-1 -> ESP32-S3-WROOM-1-N8R8; DigiKey (none) -> https://www.digikey.com/en/products/detail/espressif-system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; DigiKey Part (none) -> 5407-ESP32-S3-WROOM-1-N8R8CT-ND; ID ESP32_1 -> ESP32
- U208: renamed from U201; DigiKey (none) -> https://www.digikey.com/en/products/detail/texas-instrument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; DigiKey Part (none) -> 296-THVD1400DRCT-ND
Connections:
- net +3V3: now also C204.1, C205.1, C207.1, C209.1, C211.1, C216.1, RN201.1 (4), RN201.2, RN201.3, RN201.4, U203.8 (VCC), U205.14 (VCC), U207.8 (VCC)
- net BATT_IN: now also C202.1, L201.1, U206.1 (SW)
- net GND: now also J201.S1 (M), J201.S2 (M), C201.2, C202.2, C204.2, C205.2, C207.2, C209.2, C211.2, C212.2, C213.2, C214.2, C215.2, C216.2, R202.2, RN202.5, RN202.6, RN202.7 (5), RN202.8, U203.4 (GND), U205.7 (GND), U206.2 (GND)
- net PROG_PWR_IN: now also C201.1
- net at J201.1 (LEDA): now also C213.1, C215.1, U206.5 (V_{OUT})
- net at J201.2 (LEDK): now also J201.3 (LEDK), R202.1, U206.3 (FB)
- net FRAME_SYNC renamed FRAME_SYNC_IN
- net LCD_SPI_CS renamed SPI_CS0
- net SPI_CS0: now also U203.1 (A); no longer J201.11 (CS)
- net LCD_SPI_MOSI renamed SPI_MOSI
- net SPI_MOSI: now also U205.5 (A2), U207.5 (DI/IO_{0})
- net LCD_SPI_SCK renamed SPI_SCK
- net SPI_SCK: now also U205.9 (A3), U207.6 (CLK)
- net STRAP_GPIO45 renamed SPI_MISO
- net SPI_MISO: now also U205.3 (B1), U207.2 (DO/IO_{1})
- net STRAP_GPIO46 renamed SPI_CS1
- net SPI_CS1: now also U203.2 (B)
- new net: D202.1 (K), RN202.1 (4)
- new net: D205.1 (K), RN202.4
- new net: D204.1 (K), RN202.3
- new net: D203.1 (K), RN202.2
- new net: C212.1, C214.1, L201.2, U206.6 (V_{IN})
- new net BACKLIGHT_PWM_IN: U206.4 (CTRL)
- new net SPI_CS_FLASH: D204.2 (A), RN201.6, U203.6 (Y1), U207.1 (~{CS})
- new net SPI_CS_LCD: D205.2 (A), J201.11 (CS), RN201.5, U203.7 (Y0)
- new net SPI_CS_µSD: D203.2 (A), RN201.7 (5), U203.5 (Y2), U205.11 (B4), U205.12 (A4)
- new net SPI_MISO_µSD: U205.2 (A1)
- new net SPI_MOSI_µSD: U205.6 (B2)
- new net SPI_SCK_µSD: U205.8 (B3)
- new net SPI_µSD_BUS_CONNECT: D202.2 (A), RN201.8, U203.3 (Y3), U205.1 (1~{OE}), U205.10 (3~{OE}), U205.13 (4~{OE}), U205.4 (2~{OE})
- no-connect marks 0 -> 1
Other:
- note added: "Italics denote bootstrapping pins which go to weird states upon ESP32 reset. Be aware that these might be weird to get configured in software."
- moved on the sheet: U208
