File: Hardware/Grad/SAMD21.kicad_sch (KiCad schematic)
At the start: 19 parts, among them J1101 JST-PH SPI, J1102 JST-PH UART/I2C, J1103 JST-PH A#, J1104 Micro_SD_Card, U1101 TC7MBL3126CFT, U1102 AZ1117-5.0, U1103 THVD1400D, U1104 QTPy SAMD21

Commit message: Prototype of PCB layout
Parts:
- removed C1101, C1104, C1105: 100nF, Capacitor_SMD:C_0402_1005Metric, symbol Device:C_Small_US
- removed C1102, C1103, C1106: 22uF, Capacitor_SMD:C_0603_1608Metric, symbol Device:C_Polarized_Small_US
- removed D1101, D1102: LED_Small, New_Library:Worthington_LED_0603, symbol Device:LED_Small
- removed J1101: JST-PH SPI, Connector_JST:JST_PH_S5B-PH-K_1x05_P2.00mm_Horizontal, symbol Connector_Generic:Conn_01x05
- removed J1102: JST-PH UART/I2C, Connector_JST:JST_PH_S6B-PH-K_1x06_P2.00mm_Horizontal, symbol Connector_Generic:Conn_01x06
- removed J1103: JST-PH A#, Connector_JST:JST_PH_S6B-PH-K_1x06_P2.00mm_Horizontal, symbol Connector_Generic:Conn_01x06
- removed J1104: Micro_SD_Card, New_Library:CUI_MSD-4-A, symbol Connector:Micro_SD_Card
- removed R1101: 1k, New_Library:Worthington_R_0402, symbol Device:R_Small_US
- removed R1102: 430, New_Library:Worthington_R_0402, symbol Device:R_Small_US
- removed RN1101: 47k, New_Library:RESCAXE80P320X160X70-8N, symbol Libraries:R_Network04_Split
- removed U1101: TC7MBL3126CFT, Package_SO:TSSOP-14_4.4x5mm_P0.65mm, symbol Analog_Switch:CD4066BPW
- removed U1102: AZ1117-5.0, Package_TO_SOT_SMD:SOT-223-3_TabPin2, symbol Regulator_Linear:AZ1117-5.0
- removed U1103: THVD1400D, Package_SO:SOIC-8_3.9x4.9mm_P1.27mm, symbol Interface_UART:THVD1400D
- removed U1104: QTPy SAMD21, New_Library:Py_QT_SAMD21, symbol New_Library:QT_Py_SAMD21
Other:
- note removed: "QTPy SAMD21 has +5V -> +3V3 Regulator Onboard "3V" Pin is the output from this regulator"
